File: KiCad/KiCad.kicad_sch (KiCad schematic)
At the start: 0 parts

Commit message: KiCad Servo Driver Updates
Other:
- sheet 01_POWER: file 01power.kicad_sch -> sch/01power.kicad_sch
- sheet 02_MASTER_CONTROLLER: file 02masterController.kicad_sch -> sch/02masterController.kicad_sch
- sheet 03_SERVO_DRIVER: file 03servoDriver.kicad_sch -> sch/03servoDriver.kicad_sch
- sheet 06_DIGITAL_IO: file 06digital_IO.kicad_sch -> sch/06digital_IO.kicad_sch
- sheet 09_SAFETY: file 09safety.kicad_sch -> sch/09safety.kicad_sch
Changed lines of the file:
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@@
 			)
 		)
-		(property "Sheetfile" "09safety.kicad_sch"
+		(property "Sheetfile" "sch/09safety.kicad_sch"
 			(at 111.76 104.7246 0)
 			(show_name no)
@@
 			)
 		)
-		(property "Sheetfile" "02masterController.kicad_sch"
+		(property "Sheetfile" "sch/02masterController.kicad_sch"
 			(at 63.5 112.3446 0)
 			(show_name no)
@@
 			)
 		)
-		(property "Sheetfile" "03servoDriver.kicad_sch"
+		(property "Sheetfile" "sch/03servoDriver.kicad_sch"
 			(at 109.22 39.9546 0)
 			(show_name no)
@@
 			)
 		)
-		(property "Sheetfile" "01power.kicad_sch"
+		(property "Sheetfile" "sch/01power.kicad_sch"
 			(at 29.21 113.6146 0)
 			(show_name no)
@@
 			)
 		)
-		(property "Sheetfile" "06digital_IO.kicad_sch"
+		(property "Sheetfile" "sch/06digital_IO.kicad_sch"
 			(at 109.22 64.0846 0)
 			(show_name no)
