File: KiCad/sch/06digital_IO.kicad_sch (KiCad schematic)
At the start: 0 parts

Commit message: KiCad Servo Driver Updates
Other:
- sheet 07_LIMIT_HOME: file 07limitHome.kicad_sch -> sch/07limitHome.kicad_sch
Changed lines of the file:
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@@
 			)
 		)
-		(property "Sheetfile" "07limitHome.kicad_sch"
+		(property "Sheetfile" "sch/07limitHome.kicad_sch"
 			(at 0.0762 24.6326 0)
 			(show_name no)
@@
 		)
 		(instances
-			(project "KiCad"
-				(path "/c15a5ead-c9b6-4302-96cb-0cea8ac8d91c"
-					(page "6")
+			(project ""
+				(path "/512f3945-676f-4dfb-afc3-4a82ab9dfae9"
+					(page "")
 				)
 			)
+			(project "KiCad"
+				(path "/c15a5ead-c9b6-4302-96cb-0cea8ac8d91c/512f3945-676f-4dfb-afc3-4a82ab9dfae9"
+					(page "9")
+				)
+			)
