File: Circuits/motorDriver/PCB/motorDriver/motorDriver.kicad_sch (KiCad schematic)
At the start: 6 parts, among them J1 Conn_01x04_Pin, U1 MAX485E

Commit message: Circuits Directory
Parts:
- removed J1: Conn_01x04_Pin, symbol Connector:Conn_01x04_Pin
- added A1: Pololu_Breakout_DRV8825, Module:Pololu_Breakout-16_15.2x20.3mm, symbol Driver_Motor:Pololu_Breakout_DRV8825
Connections:
- net GND renamed GND_LOGIC
- net LOGIC_J1 renamed LOGIC_5V
- new net MOTOR_PWR: A1.8 (VMOT)
- no-connect marks 19 -> 21
Other:
- note removed: "Enkoder Pinleri"
