File: Circuits/Schematics/motorDriver/motorDriver.kicad_pcb (KiCad board)
At the start: 2 copper layers, 60 x 60 mm, 10 parts, among them J1 Conn_01x04_Pin, J2 Conn_01x02_Pin, J3 Conn_01x03_Pin, U1 MAX485E

Commit message: PSU Sim Template, Motor Driver PCB v2
Parts:
- added C3: 100nF, Capacitor_SMD:C_0805_2012Metric_Pad1.18x1.45mm_HandSolder, F.Cu at (134.3, 50.1)
- moved C2 35.1 mm to (114.6, 45.1), turned to 0 degrees
- moved R1 33.7 mm to (87.2, 61.6), turned to 180 degrees
- moved C1 33.0 mm to (114.7, 42.2), turned to 0 degrees
- moved C4 7.85 mm to (128.2, 43.3), turned to 0 degrees
Routing:
- net Net-(A2-D5): track 47.2 -> 22.8 mm
- net +5V: track 84.4 -> 61.8 mm, vias 0 -> 1
- net GND: track 102.4 -> 124.8 mm, vias 2 -> 0
- net VMOT: track 26.3 -> 29.5 mm
