File: Circuits/Schematics/masterController/masterController.kicad_pcb (KiCad board)
At the start: 2 copper layers, 37 parts, among them J1 Conn_02x03_Counter_Clockwise, J2 Screw_Terminal_01x02, J3 Screw_Terminal_01x05, J4 Screw_Terminal_01x02, K1 Relay_SPDT, SW1 SW_Push, U1 STM32F411CEUx, U2 LM2596S-ADJ, U3 AMS1117-3.3, U4 MAX485E

Commit message: Main Controller PCB Completed
Parts:
- removed J3: Screw_Terminal_01x05, TerminalBlock_Phoenix:TerminalBlock_Phoenix_PT-1,5-5-5.0-H_1x05_P5.00mm_Horizontal
- added J5: Screw_Terminal_01x02, TerminalBlock_Phoenix:TerminalBlock_Phoenix_PT-1,5-2-5.0-H_1x02_P5.00mm_Horizontal, F.Cu at (76.0, 37.5)
- added J6: Screw_Terminal_01x03, TerminalBlock_Phoenix:TerminalBlock_Phoenix_PT-1,5-3-5.0-H_1x03_P5.00mm_Horizontal, F.Cu at (115.6, 41.0)
- added R8: 120, Resistor_SMD:R_0805_2012Metric_Pad1.20x1.40mm_HandSolder, F.Cu at (122.5, 33.5)
- C14, C16: footprint Capacitor_SMD:C_Elec_10x10.2 -> Capacitor_THT:CP_Radial_D10.0mm_P5.00mm
- F1, F2: value 5A -> 35A; footprint Fuse:Fuseholder_Cylinder-5x20mm_Schurter_0031_8201_Horizontal_Open -> LebowskiBotCustomLibrary:HT-01-A
- R6: value 1k / 1W -> 10k; footprint Resistor_SMD:R_2512_6332Metric -> Resistor_SMD:R_0805_2012Metric_Pad1.20x1.40mm_HandSolder
- R7: value 120 -> 1k / 1W; footprint Resistor_SMD:R_0805_2012Metric_Pad1.20x1.40mm_HandSolder -> Resistor_SMD:R_2512_6332Metric
- moved J4 132.6 mm to (62.4, 37.5)
- moved R7 105.4 mm to (87.6, 66.2), turned to 90 degrees
- moved J2 97.4 mm to (80.8, 65.0), turned to 180 degrees
- moved R6 96.5 mm to (127.3, 29.7)
- moved U4 92.3 mm to (127.3, 33.4), turned to 180 degrees
- moved C15 91.2 mm to (127.3, 37.2)
- moved J1 83.7 mm to (144.8, 28.5), turned to -90 degrees
- moved C10 79.1 mm to (145.2, 37.9), turned to -90 degrees
- moved D1 77.3 mm to (109.7, 82.3), turned to -90 degrees
- moved F1 75.0 mm to (64.6, 63.2), turned to -90 degrees
- moved R2 71.7 mm to (144.4, 41.0), turned to 180 degrees
- moved R1 69.8 mm to (150.6, 36.8)
- moved C13 68.9 mm to (149.2, 50.3), turned to 180 degrees
- moved C9 68.6 mm to (133.5, 50.3)
- moved C1 65.4 mm to (116.3, 53.7), turned to 90 degrees
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Connections:
- C10 pad 1: GND -> GNDL
- C11 pad 1: GND -> GNDL
- C12 pad 2: GND -> GNDL
- C13 pad 1: GND -> GNDL
- C15 pad 2: GND -> GNDL
- C2 pad 1: GND -> GNDL
- C3 pad 1: GND -> GNDL
- C4 pad 1: GND -> GNDL
- C6 pad 1: GND -> GNDL
- C7 pad 1: GND -> GNDL
- C8 pad 2: GND -> GNDL
- C9 pad 1: GND -> GNDL
- J1 pad 2: GND -> GNDL
- J1 pad 5: /SWCLK -> /SWDIO
- J1 pad 6: /SWDIO -> /SWCLK
- R1 pad 1: GND -> GNDL
- R2 pad 1: GND -> GNDL
- R4 pad 1: GND -> GNDL
- R6 pad 1: Net-(K1-Pad12) -> GNDL
- R6 pad 2: GND -> Net-(U4-~{RE})
- R7 pad 1: /RS-485 A -> Net-(K1-Pad12)
- R7 pad 2: /RS-485 B -> GND
- U1 pad 10: unconnected-(U1-PA0-Pad10) -> /RS485_DE
- U1 pad 23: GND -> GNDL
- U1 pad 35: GND -> GNDL
- U1 pad 47: GND -> GNDL
- U1 pad 49: GND -> GNDL
- U1 pad 8: GND -> GNDL
- U3 pad 1: GND -> GNDL
- U4 pad 2: /RS485_RE_DE -> Net-(U4-~{RE})
- U4 pad 3: /RS485_RE_DE -> /RS485_DE
- U4 pad 5: GND -> GNDL
Routing:
- net GND: track 0.00 -> 196.5 mm
- net GNDL: track 0.00 -> 149.9 mm, vias 0 -> 3
- net +3.3V: track 0.00 -> 113.2 mm, vias 0 -> 2
- net /VIN_SECURE: track 0.00 -> 96.2 mm
- net +5V: track 0.00 -> 85.1 mm, vias 0 -> 1
- net Net-(F1-Pad2): track 0.00 -> 73.1 mm
- net /SWDIO: track 0.00 -> 42.1 mm, vias 0 -> 1
- net /SWO: track 0.00 -> 39.8 mm, vias 0 -> 1
- net /SWCLK: track 0.00 -> 37.7 mm, vias 0 -> 1
- net /NRST: track 0.00 -> 35.1 mm, vias 0 -> 1
- net VDD: track 0.00 -> 28.3 mm
- net Net-(J2-Pin_1): track 0.00 -> 27.0 mm
- net /RS485_DE: track 0.00 -> 24.5 mm, vias 0 -> 2
- net /RS485_TX: track 0.00 -> 24.4 mm, vias 0 -> 2
- net Net-(U1-BOOT0): track 0.00 -> 22.9 mm, vias 0 -> 1
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Other:
- board outline added: 111 x 71.2 mm
- board text added: "+5V A B"
- board text added: "Bot"
- board text added: "E-Stop"
- board text added: "GND VIN"
- board text added: "Lebowski"
- board text added: "VDD GND"
